File: Hardware/ir4stm32.kicad_pcb (KiCad board)
At the start: 2 copper layers, 81 x 52 mm, 76 parts, among them P1 + - R T, Q1 SS8050, Q2 SS8050, Q3 SS8050, Q4 SS8050, Q5 SS8050, Q6 SS8050, Q7 SS8050, Q8 SS8050, U1 XC6206P332MR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

Commit message: fix: (BOM)
Parts:
- R25, R26, R27, R28: value (none) -> 1K
Changed lines of the file:
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@@
   (general
     (links 144)
-    (no_connects 4)
+    (no_connects 0)
     (area 113.881 84.5876 202.850001 137.075001)
     (thickness 1.6)
@@
       (effects (font (size 1 1) (thickness 0.15)))
     )
-    (fp_text value "" (at 0 1.9 180) (layer F.Fab)
+    (fp_text value 1K (at -2.325 0 180) (layer F.Fab)
       (effects (font (size 1 1) (thickness 0.15)))
     )
@@
       (effects (font (size 1 1) (thickness 0.15)))
     )
-    (fp_text value "" (at 0 1.9 180) (layer F.Fab)
+    (fp_text value 1K (at -2.275 0 180) (layer F.Fab)
       (effects (font (size 1 1) (thickness 0.15)))
     )
@@
       (effects (font (size 1 1) (thickness 0.15)))
     )
-    (fp_text value "" (at 0 1.9 180) (layer F.Fab)
+    (fp_text value 1K (at -2.225 0 180) (layer F.Fab)
       (effects (font (size 1 1) (thickness 0.15)))
     )
@@
       (effects (font (size 1 1) (thickness 0.15)))
     )
-    (fp_text value "" (at 0 1.9 180) (layer F.Fab)
-      (effects (font (size 1 1) (thickness 0.15)))
-    )
+    (fp_text value 1K (at -2.125 0.65 180) (layer F.Fab)
+      (effects (font (size 1 1) (thickness 0.15)))
+    )
